File: Design Files/keypad/numpad-1.0.kicad_pcb (KiCad board)
At the start: 2 copper layers, 77.5 x 99.1 mm, 72 parts, among them J1 Conn_02x03_Odd_Even, J2 Conn_01x03, J3 Conn_01x03, J4 Conn_01x03, J5 Conn_01x03, J6 Conn_01x03, Q1 MOSFET-NCH-FDS6630A, SW1 KEYSW_LED, SW10 KEYSW_LED, SW11 KEYSW_LED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

Commit message: A lot of updates
Routing:
- net VCC: track 0.00 -> 434.0 mm, vias 0 -> 1
- net LED_GND: track 0.00 -> 390.4 mm, vias 0 -> 1
- net GND: track 0.00 -> 187.3 mm, vias 0 -> 1
- net ROW_5: track 0.00 -> 127.8 mm
- net COL_4: track 0.00 -> 124.5 mm
- net ROW_4: track 0.00 -> 114.6 mm
- net COL_1: track 0.00 -> 109.4 mm
- net COL_3: track 0.00 -> 106.4 mm
- net ROW_3: track 0.00 -> 94.5 mm, vias 0 -> 1
- net NEOPIXEL_CTRL: track 0.00 -> 92.2 mm, vias 0 -> 3
- net COL_2: track 0.00 -> 89.3 mm
- net ROW_2: track 0.00 -> 81.1 mm
- net A2: track 0.00 -> 71.0 mm, vias 0 -> 2
- net A3: track 0.00 -> 68.4 mm, vias 0 -> 1
- net ROW_1: track 0.00 -> 64.2 mm
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