File: Design Files/keypad/numpad.sch (KiCad schematic (older format))
At the start: 71 parts, among them J1 Conn_02x03_Odd_Even, J2 Conn_01x03, J3 Conn_01x03, J4 Conn_01x03, J5 Conn_01x03, J6 Conn_01x03, Q1 MOSFET-NCH-FDS6630A, SW1 KEYSW_LED, SW10 KEYSW_LED, SW11 KEYSW_LED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

Commit message: A lot of updates
Parts:
- SW1, SW10, SW11, SW12, SW13, SW14, SW15, SW16, SW17, SW18, SW19, SW2, SW20, SW3, SW4, SW5, SW6, SW7, SW8, SW9: symbol libkeyswitch-1_0_0:KEYSW_LED -> numpad-rescue:KEYSW_LED-libkeyswitch-1_0_0
Other:
- note added: "ATMega32u4 Pinouts \n(For use with QMK and Keyboard Firmware Builder)\n\nCols:\n- PD3, PD2, PD1, PD0\n\nRows:\n- PD4, PC6, PD7, PE6, PB4\n\nBacklight:\n- PB5\n\nNeopixel Strip:\n- PB6"
- note added: "Numpad"
Changed lines of the file:
@@
 EESchema Schematic File Version 4
-LIBS:numpad-cache
 EELAYER 30 0
 EELAYER END
@@
 $EndComp
 $Comp
-L libkeyswitch-1_0_0:KEYSW_LED SW1
+L numpad-rescue:KEYSW_LED-libkeyswitch-1_0_0 SW1
 U 1 1 5D268CF4
 P 7250 1600
@@
 $EndComp
 $Comp
-L libkeyswitch-1_0_0:KEYSW_LED SW2
+L numpad-rescue:KEYSW_LED-libkeyswitch-1_0_0 SW2
 U 1 1 5D4EE477
 P 8150 1600
@@
 $EndComp
 $Comp
-L libkeyswitch-1_0_0:KEYSW_LED SW3
+L numpad-rescue:KEYSW_LED-libkeyswitch-1_0_0 SW3
 U 1 1 5D4F2A41
 P 9050 1600
@@
 $EndComp
 $Comp
-L libkeyswitch-1_0_0:KEYSW_LED SW4
+L numpad-rescue:KEYSW_LED-libkeyswitch-1_0_0 SW4
 U 1 1 5D4F2A5A
 P 9950 1600
@@
 $EndComp
 $Comp
-L libkeyswitch-1_0_0:KEYSW_LED SW5
+L numpad-rescue:KEYSW_LED-libkeyswitch-1_0_0 SW5
 U 1 1 5D50A70C
 P 7250 2550
@@
 $EndComp
 $Comp
-L libkeyswitch-1_0_0:KEYSW_LED SW6
+L numpad-rescue:KEYSW_LED-libkeyswitch-1_0_0 SW6
 U 1 1 5D50A725
 P 8150 2550
@@
 $EndComp
 $Comp
-L libkeyswitch-1_0_0:KEYSW_LED SW7
+L numpad-rescue:KEYSW_LED-libkeyswitch-1_0_0 SW7
 U 1 1 5D50A73E
 P 9050 2550
@@
 $EndComp
 $Comp
-L libkeyswitch-1_0_0:KEYSW_LED SW8
+L numpad-rescue:KEYSW_LED-libkeyswitch-1_0_0 SW8
 U 1 1 5D50A757
 P 9950 2550
@@
 $EndComp
 $Comp
-L libkeyswitch-1_0_0:KEYSW_LED SW9
+L numpad-rescue:KEYSW_LED-libkeyswitch-1_0_0 SW9
 U 1 1 5D51F45C
 P 7250 3500
@@
 $EndComp
 $Comp
-L libkeyswitch-1_0_0:KEYSW_LED SW10
+L numpad-rescue:KEYSW_LED-libkeyswitch-1_0_0 SW10
 U 1 1 5D51F475
 P 8150 3500
@@
 $EndComp
 $Comp
-L libkeyswitch-1_0_0:KEYSW_LED SW11
+L numpad-rescue:KEYSW_LED-libkeyswitch-1_0_0 SW11
 U 1 1 5D51F48E
 P 9050 3500
@@
 $EndComp
 $Comp
-L libkeyswitch-1_0_0:KEYSW_LED SW12
+L numpad-rescue:KEYSW_LED-libkeyswitch-1_0_0 SW12
 U 1 1 5D51F4A7
 P 9950 3500
@@
 $EndComp
 $Comp
-L libkeyswitch-1_0_0:KEYSW_LED SW13
+L numpad-rescue:KEYSW_LED-libkeyswitch-1_0_0 SW13
 U 1 1 5D51F4D6
 P 7250 4450
@@
 $EndComp
 $Comp
-L libkeyswitch-1_0_0:KEYSW_LED SW14
+L numpad-rescue:KEYSW_LED-libkeyswitch-1_0_0 SW14
 U 1 1 5D51F4EF
 P 8150 4450
@@
 $EndComp
 $Comp
-L libkeyswitch-1_0_0:KEYSW_LED SW15
+L numpad-rescue:KEYSW_LED-libkeyswitch-1_0_0 SW15
 U 1 1 5D51F508
 P 9050 4450
@@
 $EndComp
 $Comp
-L libkeyswitch-1_0_0:KEYSW_LED SW16
+L numpad-rescue:KEYSW_LED-libkeyswitch-1_0_0 SW16
 U 1 1 5D51F521
 P 9950 4450
@@
 $EndComp
 $Comp
-L libkeyswitch-1_0_0:KEYSW_LED SW17
+L numpad-rescue:KEYSW_LED-libkeyswitch-1_0_0 SW17
 U 1 1 5D53AD04
 P 7250 5400
@@
 $EndComp
 $Comp
-L libkeyswitch-1_0_0:KEYSW_LED SW18
+L numpad-rescue:KEYSW_LED-libkeyswitch-1_0_0 SW18
 U 1 1 5D53AD1D
 P 8150 5400
@@
 $EndComp
 $Comp
-L libkeyswitch-1_0_0:KEYSW_LED SW19
+L numpad-rescue:KEYSW_LED-libkeyswitch-1_0_0 SW19
 U 1 1 5D53AD36
 P 9050 5400
@@
 $EndComp
 $Comp
-L libkeyswitch-1_0_0:KEYSW_LED SW20
+L numpad-rescue:KEYSW_LED-libkeyswitch-1_0_0 SW20
 U 1 1 5D53AD4F
 P 9950 5400
@@
 Text Notes 8350 6300 0    50   ~ 0
 Key Matrix and Backlighting
+Text Notes 650  2050 0    50   ~ 0
+ATMega32u4 Pinouts \n(For use with QMK and Keyboard Firmware Builder)\n\nCols:\n- PD3, PD2, PD1, PD0\n\nRows:\n- PD4, PC6, PD7, PE6, PB4\n\nBacklight:\n- PB5\n\nNeopixel Strip:\n- PB6
+Text Notes 650  850  0    100  ~ 20
+Numpad
 $EndSCHEMATC
